File: nene.kicad_pcb (KiCad board)
At the start: 2 copper layers, 81.8 x 38.1 mm, 24 parts, among them SW1 SW_Push, U1 ATmega32U4-AU, Y1 16MHz

Commit message: route and fill
Parts:
- moved C4 1.37 mm to (49.3, 118.5)
- moved R1 1.37 mm to (46.0, 118.5)
- moved USB1 0.10 mm to (35.8, 109.7)
Routing:
- net +5V: track 101.7 -> 104.2 mm
- net Net-(R1-Pad2): track 32.0 -> 33.4 mm
- net D+: track 8.62 -> 7.47 mm
- added copper zone on B.Cu, net GND
